File: diodi_small/diodi_small.sch (KiCad schematic (older format))
At the start: 10 parts, among them J1 CONN_01X04, J2 CONN_01X04

Commit message: Add files via upload
New traces and updated labels
Connections:
- net at D5.1 (K), D7.2 (A): now also J1.4 (P4); no longer J1.1 (P1)
- net at D1.2 (A), D3.1 (K): now also J1.1 (P1); no longer J1.4 (P4)
- net at D2.1 (K), D4.2 (A): now also J2.4 (P4); no longer J2.1 (P1)
- net at D6.2 (A), D8.1 (K): now also J2.1 (P1); no longer J2.4 (P4)
Changed lines of the file:
@@
 F 3 "" H 2750 2200 50  0001 C CNN
 	1    2750 2200
-	-1   0    0    1
+	-1   0    0    -1
 $EndComp
 $Comp
@@
 F 3 "" H 4450 2200 50  0001 C CNN
 	1    4450 2200
-	1    0    0    -1
+	1    0    0    1
 $EndComp
 $Comp
@@
 	3050 2050 2950 2050
 Wire Wire Line
-	3100 1800 3050 1800
-Connection ~ 3050 1900
+	2950 1800 3100 1800
 Wire Wire Line
-	3850 1800 4200 1800
+	3850 1800 4250 1800
 Wire Wire Line
 	4200 1800 4200 2050
@@
 Wire Wire Line
 	4200 2050 4250 2050
-Connection ~ 4200 1900
 $Comp
 L D D7
@@
 	3050 2350 2950 2350
 Wire Wire Line
-	3100 2600 3050 2600
-Connection ~ 3050 2500
+	2950 2600 3100 2600
 Wire Wire Line
-	3850 2600 4200 2600
+	3850 2600 4250 2600
 Wire Wire Line
 	4200 2600 4200 2350
@@
 Wire Wire Line
 	4200 2350 4250 2350
-Connection ~ 4200 2500
 Wire Wire Line
 	4250 2150 2950 2150
 Wire Wire Line
 	2950 2250 4250 2250
+Connection ~ 3050 1900
+Connection ~ 4200 1900
+Connection ~ 4200 2500
+Connection ~ 3050 2500
+Wire Wire Line
+	2950 2050 2950 1800
+Connection ~ 3050 1800
+Wire Wire Line
+	4250 2050 4250 1800
+Connection ~ 4200 1800
+Wire Wire Line
+	2950 2350 2950 2600
+Connection ~ 3050 2600
+Wire Wire Line
+	4250 2350 4250 2600
+Connection ~ 4200 2600
 $EndSCHEMATC

Commit message: Add files via upload
Other:
- note added: "All credits to Addictivers.cc"
- note added: "CERN OSH License 1.2"
- note added: "Stepper_motor_lifeguard_V2"
Changed lines of the file:
@@
 	4250 2350 4250 2600
 Connection ~ 4200 2600
+Text Notes 7350 7500 0    60   ~ 0
+Stepper_motor_lifeguard_V2
+Text Notes 7100 6750 0    60   ~ 0
+CERN OSH License 1.2
+Text Notes 7100 6900 0    60   ~ 0
+All credits to Addictivers.cc
 $EndSCHEMATC
